File: eagle/vc_pan.brd (EAGLE design)
At the start: 100 x 80 mm, 49 parts, among them IC1 TL074P, IC2 LM13700N, IC3 TL072P, Q1 2N3906, Q2 2N3906

Commit message: 85 percentish routed
Parts:
- moved U$2 159.1 mm to (76.2, 17.8), turned to 90 degrees
- moved C10 140.5 mm to (66.0, 16.5), turned to 270 degrees
- moved C2 139.1 mm to (72.4, 17.8), turned to 270 degrees
- moved PWR1 138.5 mm to (64.8, 6.35), turned to 180 degrees
- moved U$1 133.0 mm to (58.4, 16.5), turned to 90 degrees
- moved C1 119.3 mm to (62.2, 16.5), turned to 270 degrees
- moved C9 117.3 mm to (53.3, 31.8), turned to 90 degrees
- moved C5 106.4 mm to (68.6, 16.5), turned to 90 degrees
- moved C8 96.6 mm to (30.5, 6.35), turned to 180 degrees
- moved C7 82.6 mm to (35.6, 52.1)
- moved C6 77.3 mm to (30.5, 19.1), turned to 180 degrees
- moved C4 55.9 mm to (27.9, 31.8), turned to 90 degrees
- moved C3 46.2 mm to (27.9, 64.8), turned to 90 degrees
- moved R1 5.08 mm to (22.9, 69.8), turned to 180 degrees
- moved R10 4.02 mm to (36.8, 22.9)
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Routing:
- net GND: track 0.00 -> 342.0 mm
- net -12V: track 0.00 -> 312.6 mm
- net N$6: track 0.00 -> 130.7 mm
- net +12V: track 0.00 -> 127.1 mm
- net N$21: track 0.00 -> 62.3 mm
- net N$18: track 0.00 -> 29.9 mm
- net N$2: track 0.00 -> 25.8 mm
- net N$13: track 0.00 -> 25.7 mm
- net N$22: track 0.00 -> 25.4 mm
- net N$8: track 0.00 -> 23.9 mm
- net N$5: track 0.00 -> 22.4 mm
- net N$11: track 0.00 -> 20.8 mm
- net N$30: track 0.00 -> 20.5 mm
- net N$19: track 0.00 -> 17.5 mm
- net N$20: track 0.00 -> 17.1 mm
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